File: rgbled-controller.kicad_sch (KiCad schematic)
At the start: 21 parts, among them IC1 ME6211C33M5G-N, J1 PROG_HDR, J2 IC2_Header, J3 Power In, J4 LED_OUT, Q1 UMH3N, Q2 2N7002, SW1 SW_Reset, SW2 SW_Flash, U1 ESP-12F

Commit message: changed board layout and added spare pins
Parts:
- added TP1: LED_CTRL, TestPoint:TestPoint_Pad_2.0x2.0mm, symbol Connector:TestPoint
- J2: footprint Connector_IDC:IDC-Header_2x03_P2.54mm_Vertical -> Chof747 Connectors:HDR-TH_6P-P2.54-V-F-R2-C3-S2.54-4
- SW1: value SW_Reset -> Reset
- SW2: value SW_Flash -> Flash
Connections:
- net GPIO2_LED_CTRL: now also TP1.1
Changed lines of the file:
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@@
 	(wire
 		(pts
+			(xy 187.96 160.02) (xy 191.77 160.02)
+		)
+		(stroke
+			(width 0)
+			(type default)
+		)
+	)
+	(wire
+		(pts
 			(xy 208.28 82.55) (xy 214.63 82.55)
 		)
@@
 		)
 	)
+	(hierarchical_label "GPIO2_LED_CTRL"
+		(shape input)
+		(at 187.96 160.02 180)
+		(effects
+			(font
+				(size 1.27 1.27)
+			)
+			(justify right)
+		)
+	)
 	(hierarchical_label "~{GPIO0_INT_FLASH}"
 		(shape input)
@@
 			)
 		)
-		(property "Value" "SW_Reset"
+		(property "Value" "Reset"
 			(at 119.38 168.9099 90)
 			(effects
@@
 			)
 		)
-		(property "Footprint" "Connector_IDC:IDC-Header_2x03_P2.54mm_Vertical"
+		(property "Footprint" "Chof747 Connectors:HDR-TH_6P-P2.54-V-F-R2-C3-S2.54-4"
 			(at 219.71 80.01 0)
 			(effects
@@
 			)
 		)
-		(property "Value" "SW_Flash"
+		(property "Value" "Flash"
 			(at 156.21 168.9099 90)
 			(effects
@@
 					(unit 1)
 				)
+			)
+		)
+	)
+	(symbol
+		(lib_id "Connector:TestPoint")
+		(at 191.77 160.02 0)
+		(unit 1)
+		(exclude_from_sim no)
+		(in_bom yes)
+		(on_board yes)
+		(dnp no)
+		(fields_autoplaced yes)
+		(property "Reference" "TP1"
+			(at 194.31 155.4479 0)
+			(effects
+				(font
+					(size 1.27 1.27)
+				)
+				(justify left)
+			)
+		)
+		(property "Value" "LED_CTRL"
+			(at 194.31 157.9879 0)
+			(effects
+				(font
+					(size 1.27 1.27)
+				)
+				(justify left)
+			)
+		)
+		(property "Footprint" "TestPoint:TestPoint_Pad_2.0x2.0mm"
+			(at 196.85 160.02 0)
+			(effects
+				(font
+					(size 1.27 1.27)
+				)
+				(hide yes)
+			)
+		)
+		(property "Datasheet" "~"
+			(at 196.85 160.02 0)
+			(effects
+				(font
+					(size 1.27 1.27)
+				)
+				(hide yes)
+			)
+		)
+		(property "Description" "test point"
+			(at 191.77 160.02 0)
+			(effects
+				(font
+					(size 1.27 1.27)
+				)
+				(hide yes)
+			)
+		)
+		(pin "1"
+		)
+		(instances
+			(project ""
+				(path "/e8426e51-e5a9-4642-8277-6d3f50e0e523"
+					(reference "TP1")
+					(unit 1)
+				)
