File: peripheral/rgbled-peripheral.kicad_pcb (KiCad board)
At the start: 2 copper layers, 126.3 x 20 mm, 15 parts, among them J1 Spare Pins, J2 IC2_Header, SW1 Seg 1, SW2 Seg 2, SW3 Seg 3, SW4 Seg 4, SW5 Seg 5, SW6 Mod, U1 MCP23017_SO, U2 SHT4x

Commit message: initial production version
Routing:
- net +3V3: track 123.7 -> 143.2 mm, vias 2 -> 6
- net IOEXP_SDA: track 70.4 -> 69.7 mm
- net GND: vias 6 -> 7
Changed lines of the file:
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@@
 	)
 	(segment
-		(start 145.5 59.6)
-		(end 149.1 59.6)
-		(width 0.13)
-		(layer "F.Cu")
-		(net 5)
-	)
-	(segment
-		(start 149.1 59.6)
-		(end 149.77 58.93)
+		(start 142.8 56.9)
+		(end 144.9 59)
+		(width 0.13)
+		(layer "F.Cu")
+		(net 5)
+	)
+	(segment
+		(start 90.4 62.3)
+		(end 90.7 62)
+		(width 0.13)
+		(layer "F.Cu")
+		(net 5)
+	)
+	(segment
+		(start 144.9 59)
+		(end 149.2 59)
+		(width 0.13)
+		(layer "F.Cu")
+		(net 5)
+	)
+	(segment
+		(start 90.7 62)
+		(end 95.6 62)
+		(width 0.13)
+		(layer "F.Cu")
+		(net 5)
+	)
+	(segment
+		(start 104.5 56.9)
+		(end 142.8 56.9)
+		(width 0.13)
+		(layer "F.Cu")
+		(net 5)
+	)
+	(segment
+		(start 98.5 64.9)
+		(end 100.66425 64.9)
+		(width 0.13)
+		(layer "F.Cu")
+		(net 5)
+	)
+	(segment
+		(start 100.66425 64.9)
+		(end 102.26 63.30425)
 		(width 0.13)
 		(layer "F.Cu")
@@
 	)
 	(segment
-		(start 90.4 62.3)
-		(end 90.7 62)
-		(width 0.13)
-		(layer "F.Cu")
-		(net 5)
-	)
-	(segment
-		(start 104.5 56.9)
-		(end 142.8 56.9)
-		(width 0.13)
-		(layer "F.Cu")
-		(net 5)
-	)
-	(segment
-		(start 90.7 62)
-		(end 95.6 62)
-		(width 0.13)
-		(layer "F.Cu")
-		(net 5)
-	)
-	(segment
-		(start 149.77 58.93)
+		(start 149.77 58.43)
 		(end 149.77 57.37675)
 		(width 0.13)
@@
 	)
 	(segment
-		(start 98.5 64.9)
-		(end 100.66425 64.9)
+		(start 149.2 59)
+		(end 149.77 58.43)
 		(width 0.13)
 		(layer "F.Cu")
@@
 	)
 	(segment
-		(start 142.8 56.9)
-		(end 145.5 59.6)
-		(width 0.13)
-		(layer "F.Cu")
-		(net 5)
-	)
-	(segment
-		(start 100.66425 64.9)
-		(end 102.26 63.30425)
-		(width 0.13)
-		(layer "F.Cu")
-		(net 5)
-	)
-	(segment
 		(start 87 60.7375)
 		(end 87.6375 60.1)
@@
 	)
 	(segment
+		(start 107.8 61.6)
+		(end 107.8 66.699998)
+		(width 0.25)
+		(layer "F.Cu")
+		(net 6)
+	)
+	(segment
 		(start 87.7625 61.5)
 		(end 87 60.7375)
@@
 	)
 	(segment
+		(start 97.8 65.4)
+		(end 97.8 66.7)
+		(width 0.25)
+		(layer "F.Cu")
+		(net 6)
+	)
+	(segment
 		(start 100.6 53.8)
 		(end 154.8 53.8)
@@
 	)
 	(segment
+		(start 99.8 68.7)
+		(end 104.8 68.7)
+		(width 0.25)
+		(layer "F.Cu")
+		(net 6)
+	)
+	(segment
 		(start 89 61.5)
 		(end 87.7625 61.5)
@@
 	)
 	(segment
+		(start 107.8 66.699998)
+		(end 106.85 67.65)
+		(width 0.25)
+		(layer "F.Cu")
+		(net 6)
+	)
+	(segment
+		(start 99.8 68.7)
+		(end 97.8 66.7)
+		(width 0.25)
+		(layer "F.Cu")
+		(net 6)
+	)
+	(segment
 		(start 154.8 53.8)
 		(end 170.1 53.8)
@@
 		(width 0.25)
 		(layer "F.Cu")
+		(net 6)
+	)
+	(via
+		(at 97.8 65.4)
+		(size 0.8)
+		(drill 0.4)
+		(layers "F.Cu" "B.Cu")
+		(net 6)
+	)
+	(via
+		(at 107.8 61.6)
+		(size 0.8)
+		(drill 0.4)
+		(layers "F.Cu" "B.Cu")
+		(net 6)
+	)
+	(via
+		(at 104.8 68.7)
+		(size 0.8)
+		(drill 0.4)
+		(layers "F.Cu" "B.Cu")
 		(net 6)
 	)
@@
 		(net 6)
 	)
+	(via
+		(at 106.85 67.65)
+		(size 0.8)
+		(drill 0.4)
+		(layers "F.Cu" "B.Cu")
+		(net 6)
+	)
 	(segment
 		(start 88.3 60.1)
@@
 	)
 	(segment
-		(start 103.13575 59.1)
-		(end 104.8 60.76425)
-		(width 0.25)
-		(layer "B.Cu")
-		(net 6)
-	)
-	(segment
 		(start 96.95 59.15)
 		(end 97 59.1)
@@
 	)
 	(segment
+		(start 97.8 65.4)
+		(end 97.8 60)
+		(width 0.25)
+		(layer "B.Cu")
+		(net 6)
+	)
+	(segment
+		(start 105.8 68.7)
+		(end 104.8 68.7)
+		(width 0.25)
+		(layer "B.Cu")
+		(net 6)
+	)
+	(segment
+		(start 105.8 68.7)
+		(end 106.85 67.65)
+		(width 0.25)
+		(layer "B.Cu")
+		(net 6)
+	)
+	(segment
+		(start 106.96425 60.76425)
+		(end 107.8 61.6)
+		(width 0.25)
+		(layer "B.Cu")
+		(net 6)
+	)
+	(segment
+		(start 104.8 60.76425)
+		(end 106.96425 60.76425)
+		(width 0.25)
+		(layer "B.Cu")
+		(net 6)
+	)
+	(segment
 		(start 92.2 61.5)
 		(end 94.6 61.5)
@@
 	)
 	(segment
-		(start 97 59.1)
-		(end 103.13575 59.1)
+		(start 97.8 60)
+		(end 96.95 59.15)
 		(width 0.25)
 		(layer "B.Cu")
@@
 	)
 	(segment
+		(start 97.90425 63.30425)
+		(end 99.72 63.30425)
+		(width 0.13)
+		(layer "F.Cu")
+		(net 7)
+	)
+	(segment
 		(start 110.825 62.725)
 		(end 110.8 62.7)
@@
 		(end 147.32325 66.67675)
 		(width 0.25)
+		(layer "F.Cu")
+		(net 7)
+	)
+	(segment
+		(start 96.90425 62.30425)
+		(end 97.90425 63.30425)
+		(width 0.13)
 		(layer "F.Cu")
 		(net 7)
@@
 	)
 	(via
+		(at 96.90425 62.30425)
+		(size 0.5)
+		(drill 0.2)
+		(layers "F.Cu" "B.Cu")
+		(net 7)
+	)
+	(via
 		(at 153.607707 58.907707)
 		(size 0.8)
@@
 	)
 	(segment
+		(start 90.9 63.3)
+		(end 92.2 62)
+		(width 0.13)
+		(layer "B.Cu")
+		(net 7)
+	)
+	(segment
+		(start 96.6 62)
+		(end 96.90425 62.30425)
+		(width 0.13)
+		(layer "B.Cu")
+		(net 7)
+	)
+	(segment
 		(start 92.2 62)
-		(end 98.41575 62)
+		(end 96.6 62)
 		(width 0.13)
 		(layer "B.Cu")
@@
 		(width 0.13)
 		(layer "B.Cu")
-		(net 7)
-	)
-	(segment
-		(start 90.9 63.3)
-		(end 92.2 62)
-		(width 0.13)
-		(layer "B.Cu")
-		(net 7)
-	)
-	(segment
-		(start 98.41575 62)
-		(end 99.72 63.30425)
-		(width 0.13)
-		(layer "B.Cu")
