File: controller/rgbled-controller.kicad_pcb (KiCad board)
At the start: 2 copper layers, 65 x 40 mm, 26 parts, among them IC1 ME6211C33M5G-N, J1 PROG_HDR, J2 IC2_Header, J3 Power In, J4 Led Strip, J5 Power Selector, J6 3v3 Iin, Q1 UMH3N, Q2 2N7002, SW1 Reset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

Commit message: initial production version
Parts:
- removed the G*** at (30.5, 184.9)
- removed JP2: Wake enable, Jumper:SolderJumper-2_P1.3mm_Open_Pad1.0x1.5mm
- removed JX: Reserve, Connector_PinHeader_2.54mm:PinHeader_2x02_P2.54mm_Vertical
- added J7: Conn_01x02_Pin, Connector_PinHeader_2.54mm:PinHeader_1x02_P2.54mm_Vertical, F.Cu at (166.6, 84.1)
- added J8: Heater, Chof747_Connectors:CONN-TH_4P-P2.54_KF128-2.54-4P, F.Cu at (173.2, 71.7)
- added Q3: 2N7002, Package_TO_SOT_SMD:SOT-23, F.Cu at (147.1, 93.3)
- added R5: 10k, Resistor_SMD:R_0603_1608Metric_Pad0.98x0.95mm_HandSolder, F.Cu at (158.3, 93.0)
- added R6: 10k, Resistor_SMD:R_0603_1608Metric_Pad0.98x0.95mm_HandSolder, F.Cu at (125.7, 82.5)
- added R7: 10k, Resistor_SMD:R_0603_1608Metric_Pad0.98x0.95mm_HandSolder, F.Cu at (151.6, 89.3)
- added TP2: LED2, TestPoint:TestPoint_Pad_2.0x2.0mm, F.Cu at (141.4, 93.3)
- C2: value 1uF -> 10uF
- J3: value Power In -> Power In 1
- J4: value Led Strip -> Power In 2; footprint TerminalBlock:TerminalBlock_bornier-3_P5.08mm -> TerminalBlock:TerminalBlock_bornier-2_P5.08mm
- J5: value Power Selector -> Strip 2; footprint Connector_PinHeader_2.54mm:PinHeader_1x03_P2.54mm_Vertical -> TerminalBlock:TerminalBlock_bornier-3_P5.08mm
- J6: value 3v3 Iin -> Strip 1; footprint TerminalBlock:TerminalBlock_bornier-2_P5.08mm -> TerminalBlock:TerminalBlock_bornier-3_P5.08mm
- TP1: value LED_CTRL -> LED1
- moved F1 68.2 mm to (166.6, 79.8), turned to 180 degrees
- moved J1 58.9 mm to (165.6, 75.7), turned to 180 degrees
- moved Q1 54.2 mm to (160.2, 64.1), turned to 0 degrees
- moved J5 52.5 mm to (147.0, 104.5)
- moved J3 43.5 mm to (135.2, 104.5)
- moved C3 39.3 mm to (173.1, 82.5), turned to 0 degrees
- moved IC1 37.1 mm to (173.1, 86.2), turned to 90 degrees
- moved C2 35.6 mm to (173.1, 89.8), turned to 0 degrees
- moved RN1 28.0 mm to (160.3, 72.2), turned to -90 degrees
- moved C1 24.5 mm to (128.2, 82.5)
- moved U1 24.2 mm to (138.0, 71.1)
- moved R2 24.0 mm to (148.2, 80.5)
- moved SW2 23.6 mm to (115.2, 62.1), turned to 180 degrees
- moved R4 20.6 mm to (120.6, 70.5)
- moved R1 20.5 mm to (122.5, 70.5), turned to -90 degrees
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Connections:
- net /GPIO3_RX renamed GPIO3_RX
- net /GPIO4_TX renamed GPIO4_TX
- C3 pad 1: /3v3_regulator -> +3V3
- F1 pad 1: /3v3PROG_SAVE -> 3v3PROG_SAVE
- IC1 pad 5: /3v3_regulator -> +3V3
- J3 pad 1: +5V -> +5V/1
- J4 pad 1: GND -> +5V
- J4 pad 2: +5V -> GND
- J5 pad 1: /3v3PROG_SAVE -> OUT_LED_CTRL_2
- J5 pad 2: +3V3 -> GND
- J5 pad 3: /3v3_regulator -> +5V
- J6 pad 1: /3v3PROG -> OUT_LED_CTRL_1
- Q2 pad 2: /GPIO2_LED_CTRL -> GPIO12_LED_CTRL_1
- Q2 pad 3: OUT_LED_CTRL -> OUT_LED_CTRL_1
- R3 pad 2: OUT_LED_CTRL -> OUT_LED_CTRL_1
- RN1 pad 4: /GPIO2_LED_CTRL -> GPIO2_HEATER_SENSOR
- TP1 pad 1: /GPIO2_LED_CTRL -> GPIO12_LED_CTRL_1
- U1 pad 17: /GPIO2_LED_CTRL -> GPIO2_HEATER_SENSOR
- U1 pad 4: GPIO16_WAKE -> unconnected-(U1-GPIO16-Pad4)
- U1 pad 5: unconnected-(U1-GPIO14-Pad5) -> GPIO14_HEATER_LED
- U1 pad 6: unconnected-(U1-GPIO12-Pad6) -> GPIO12_LED_CTRL_1
- U1 pad 7: unconnected-(U1-GPIO13-Pad7) -> GPIO13_LED_CTRL_2
Routing:
- net +3V3: track 91.5 -> 233.0 mm, vias 4 -> 6
- net /3v3_regulator: track 63.8 -> 0.00 mm, vias 1 -> 0
- net OUT_LED_CTRL_1: track 0.00 -> 53.3 mm
- net GPIO14_HEATER_LED: track 0.00 -> 50.0 mm, vias 0 -> 4
- net ~{GPIO0_INT_FLASH}: track 69.9 -> 112.1 mm, vias 2 -> 4
- net +5V: track 12.8 -> 52.2 mm
- net Net-(U1-EN): track 42.3 -> 7.98 mm, vias 2 -> 0
- net GPIO13_LED_CTRL_2: track 0.00 -> 33.3 mm
- net GPIO2_HEATER_SENSOR: track 0.00 -> 30.8 mm, vias 0 -> 2
- net GPIO12_LED_CTRL_1: track 0.00 -> 25.5 mm
- net /GPIO2_LED_CTRL: track 24.7 -> 0.00 mm
- net OUT_LED_CTRL_2: track 0.00 -> 22.2 mm
- net ~{RESET}: track 87.1 -> 73.2 mm, vias 5 -> 2
- net OUT_LED_CTRL: track 12.9 -> 0.00 mm
- net GPIO4_TX: track 33.4 -> 20.6 mm
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- added copper zone on B.Cu, net +5V
- added copper zone on B.Cu, net +5V/1
- added copper zone on F.Cu, net +5V/1
Other:
- board size 65 x 40 mm -> 70 x 50 mm
- board text added: "DAT 1"
- board text added: "DAT 2"
- board text added: "L"
- board text added: "S"
- board text removed: "12"
- board text removed: "14"
- board text removed: "DAT"
- board text removed: "Dir"
- board text removed: "Reg"
